File: hardware/interview.kicad_sch (KiCad schematic)
At the start: 14 parts, among them U1 TPS922055DRRR, U2 STM32G031K6Tx, U3 LM2596S-3.3

Commit message: progress on hardware schematic
Parts:
- removed D1: 1N4148WT, Diode_SMD:D_SOD-523, symbol Diode:1N4148WT
- removed R4, R5: R_US, symbol Device:R_US
- removed U3: LM2596S-3.3, Package_TO_SOT_SMD:TO-263-5_TabPin3, symbol Regulator_Switching:LM2596S-3.3
- added C1: 1u, symbol Device:C_US
- added C2: 2.2u, symbol Device:C_US
- added C3: 100n, symbol Device:C_US
- added C4: 4.7u, symbol Device:C_US
- added C5, C_in, C_out_2: 0.1u, symbol Device:C_US
- added C_in_1: 68u, symbol Device:C_US
- added C_out_1: 0.47u, symbol Device:C_US
- added D1: SS34, Diode_SMD:D_SMC, symbol Diode:SS34
- added J1: 12V_external_power_supply, symbol Connector:Conn_01x02_Pin
- added J2: TEC_Module_connection, symbol Connector:Conn_01x02_Pin
- added J4: Conn_01x04_Pin, symbol Connector:Conn_01x04_Pin
- added R_COMP: 100, symbol Device:R_US
- added R_balance (x2), R_boost: 10k, symbol Device:R_US
- added TH1: Thermistor_NTC_1, symbol Device:Thermistor_NTC_US
- added TH2: Thermistor_NTC_2, symbol Device:Thermistor_NTC_US
- added U3: TPS70933DRVR, DRV6_1P6X1_TEX, symbol 2026-05-04_01-50-01:TPS70933DRVR
- C_COMP: renamed from C3; value C_US -> 1n
- C_in_2: renamed from C2; value C_US -> 22u
- C_vcc: renamed from C1; value C_US -> 1u
- L1: value L -> 10uH
- R1: value R_US -> 20k
- R_FSET: renamed from R2; value R_US -> 59k
- R_RLT: renamed from R3; value R_US -> 100
- R_SENSE: renamed from R6; value R_US -> 52.5m
Connections:
- net GND: now also U2.5 (VSS), C1.2, C2.2, C3.2, C4.2, C5.2, C_in_1.2, J1.1 (Pin_1), J4.1 (Pin_1), R_balance.1, R_balance.1, R_boost.2, U3.3 (GND)
- net TEC+: now reaches C_in_2.1, U1.1 (VIN)
- net TEC+: now also C_vcc.1, U1.2 (VCC), C1.1, C_in.1, C_in.2, C_in_1.1, C_out_1.1, C_out_2.1, D1.1 (K), J1.2 (Pin_2), J2.2 (Pin_2), U3.1 (IN); no longer R_SENSE.1
- net at L1.1, U1.12 (SW): now also D1.2 (A)
- net PWM: now reaches U1.3 (ADIM/HD)
- net PWM: now also U2.18 (PA8)
- net Driver_EN: now reaches U1.4 (EN/PWM)
- net Driver_EN: now also U2.12 (PA5)
- net Driver_FAULT: now reaches U1.5 (FAULT)
- net Driver_FAULT: now also U2.13 (PA6)
- net at U1.8 (COMP): now also R_COMP.1; no longer C_COMP.1
- net TEC-: now reaches R_RLT.2
- net TEC-: now also R_SENSE.1, C_out_1.2, C_out_2.2, J2.1 (Pin_1)
- net SWDIO: now reaches U2.24 (PA13)
- net SWDIO: now also J4.3 (Pin_3)
- net SWCLK: now reaches U2.25 (PA14)
- net SWCLK: now also J4.2 (Pin_2), R_boost.1
- net VDD: now reaches U2.4 (VDD)
- net VDD: now also C2.1, C3.1, C4.1, J4.4 (Pin_4), TH1.2, TH2.2, U3.5 (OUT)
- net at U2.6 (PF2): now also C5.1
- net at U2.8 (PA1): now also R_balance.2, TH1.1
- net at U2.9 (PA2): now also R_balance.2, TH2.1
- new net: C_COMP.1, R_COMP.2
- no-connect marks 0 -> 23
Other:
- note added: "Active_High"
- note added: "Actuator: PWM controlled TEC driver (0-4A)"
- note added: "External Power Supply"
- note added: "MCU Power Management to 3.3V"
- note added: "MCU controller"
- note added: "Normally_Low"
- note added: "PWM signal"
- note added: "TEC connector"
- note added: "Thermal Feedback Sensing"
- note added: "boot from user flash"
- note added: "configure using internal pull up and down for GPIO"
- note added: "debugger connector"
- title: (none) -> Interview Challenge: TEC Driver Design
- moved on the sheet: C_COMP, C_in_2, C_vcc, L1, R1, R_FSET, R_RLT, R_SENSE, U1, U2
